File: NoiseMaker/NoiseMaker.sch (KiCad schematic (older format))
At the start: 20 parts, among them J1 IDE_OUT, J2 IDE_IN, J3 PWR, J4 SPK, M1 Mounting, M2 Mounting, M3 Mounting, SW1 TEST, SW2 VOL_UP, SW3 VOL_DOWN

Commit message: JP2 now THT jumper
Parts:
- JP2: footprint solder_bridge:select2 -> Connector_PinHeader_2.54mm:PinHeader_1x03_P2.54mm_Vertical
Changed lines of the file:
@@
 F 0 "JP2" H 2050 6400 50  0000 L CNN
 F 1 "DRV_SEL2" H 2050 6475 50  0000 L CNN
-F 2 "solder_bridge:select2" H 1950 6650 50  0001 C CNN
+F 2 "Connector_PinHeader_2.54mm:PinHeader_1x03_P2.54mm_Vertical" H 1950 6650 50  0001 C CNN
 F 3 "~" H 1950 6650 50  0001 C CNN
 	1    1950 6650
@@
 Wire Wire Line
 	6825 3125 6900 3125
+Connection ~ 6900 3125
+Wire Wire Line
+	6900 3125 6900 3400
 Wire Bus Line
 	1100 2075 1100 7125
@@
 Wire Bus Line
 	1400 2075 1400 4225
-Connection ~ 6900 3125
-Wire Wire Line
-	6900 3125 6900 3400
 $EndSCHEMATC

Commit message: Account for two common passive buzzers
Parts:
- LS1: footprint Buzzer_Beeper:Buzzer_12x9.5RM7.6 -> Buzzer:Buzzer_12x9.5RM7.6
Changed lines of the file:
@@
 F 0 "LS1" H 7863 3267 50  0000 C CNN
 F 1 "Speaker" H 7863 3176 50  0000 C CNN
-F 2 "Buzzer_Beeper:Buzzer_12x9.5RM7.6" H 7900 2750 50  0001 C CNN
+F 2 "Buzzer:Buzzer_12x9.5RM7.6" H 7900 2750 50  0001 C CNN
 F 3 "~" H 7890 2900 50  0001 C CNN
 	1    7900 2950

Commit message: Rename library
Parts:
- LS1: footprint Buzzer:Buzzer_12x9.5RM7.6 -> small_buzzer:Buzzer_12x9.5RM7.6
Changed lines of the file:
@@
 F 0 "LS1" H 7863 3267 50  0000 C CNN
 F 1 "Speaker" H 7863 3176 50  0000 C CNN
-F 2 "Buzzer:Buzzer_12x9.5RM7.6" H 7900 2750 50  0001 C CNN
+F 2 "small_buzzer:Buzzer_12x9.5RM7.6" H 7900 2750 50  0001 C CNN
 F 3 "~" H 7890 2900 50  0001 C CNN
 	1    7900 2950

Commit message: Update README and tweak silkscreen
Parts:
- D1: value 1n4001 -> 1N5819; symbol Device:D_Small -> Diode:1N5819
- JP1: footprint solder_bridge:select2 -> Connector_PinHeader_2.54mm:PinHeader_1x03_P2.54mm_Vertical
Changed lines of the file:
@@
 NoConn ~ 5675 2125
 $Comp
-L Device:D_Small D1
+L Diode:1N5819 D1
 U 1 1 634D2772
 P 9025 4800
 F 0 "D1" H 9025 5007 50  0000 C CNN
-F 1 "1n4001" H 9025 4916 50  0000 C CNN
+F 1 "1N5819" H 9025 4916 50  0000 C CNN
 F 2 "Diode_THT:D_DO-41_SOD81_P12.70mm_Horizontal" V 9025 4800 50  0001 C CNN
 F 3 "~" V 9025 4800 50  0001 C CNN
@@
 NoConn ~ 5475 2125
 NoConn ~ 9850 3100
-Wire Wire Line
-	8925 4800 8775 4800
 Wire Wire Line
 	8775 4800 8775 4725
@@
 F 0 "JP1" H 2050 5850 50  0000 L CNN
 F 1 "DRV_SEL1" H 2050 5925 50  0000 L CNN
-F 2 "solder_bridge:select2" H 1950 6100 50  0001 C CNN
+F 2 "Connector_PinHeader_2.54mm:PinHeader_1x03_P2.54mm_Vertical" H 1950 6100 50  0001 C CNN
 F 3 "~" H 1950 6100 50  0001 C CNN
 	1    1950 6100
@@
 Connection ~ 9250 5000
 NoConn ~ 9350 5100
-Wire Wire Line
-	9125 4800 9350 4800
 $Comp
 L Switch:SW_Push SW2
@@
 Wire Wire Line
 	6900 3125 6900 3400
+Wire Wire Line
+	8775 4800 8875 4800
+Wire Wire Line
+	9175 4800 9350 4800
 Wire Bus Line
 	1100 2075 1100 7125
